File: examples/LoRaWAN/Water_monitoring/WaterSensorNode/pcb/KijaniCarrier.kicad_pcb (KiCad board)
At the start: 2 copper layers, 100 x 100 mm, 52 parts, among them J2 SW_1, J3 ANALOG, J4 DIGITAL, J5 I2C_PORT, J6 BAT_IN, J7 SMA pH, J8 A/B, J9 SMA EC, Q1 AO3401A, Q2 2N7002, Q3 AO3401A, Q4 2N7002, U1 U3V9F12, U2 MCP1700-3302, U3 MAX3485, U4 BE-IVI pH, U5 BE-IVI EC, U6 EZO-pH, U7 EZO-EC, X1 CELL, X2 DS18B20, X3 PROBE1, X4 PROBE2

Commit message: PCB design refined, shortcomings script solved
Other:
- board text added: "18650 CELL IN"
- board text added: "A1=ISOLATORS D5=12V D6=3V3"
- board text added: "ANALOG"
- board text added: "D6- IS NOT GND - KEEP APART"
- board text added: "DIGITAL"
- board text added: "I2C_PORT"
- board text added: "ISOLATED"
- board text added: "J6 = POWER OUT TO WAZISENSE"
- board text added: "LEAVE OPEN, DO NOT BRIDGE:"
- board text added: "MODULES: PIN1 = SQUARE PAD"
- board text added: "PGND NEVER TO GND"
- board text added: "POWER_OUT"
- board text added: "R11 R12 U2 (JP1 REPLACES U2)"
- board text added: "RS485 MODULE A/B"
- board text added: "SW_1"
- board text added: "TO WAZISENSE"
- board text added: "U4A"
- board text added: "U4B"
- board text added: "U5A"
- board text added: "U5B"
- board text added: "U6A"
- board text added: "U6B"
- board text added: "U7A"
- board text added: "U7B"
- board text added: "X1 = 18650 CELL IN"
- board text removed: "A1 = ISOLATOREN EIN"
- board text removed: "D5 = 12V EIN"
- board text removed: "D6 = 3V3 EIN"
- board text removed: "ISOLIERT"
- board text removed: "J2 SW_1 J3 ANALOG"
- board text removed: "J4 DIGITAL J5 I2C"
- board text removed: "J6 BAT_IN"
- board text removed: "JP1 BESTUECKEN, U2 NICHT"
- board text removed: "MAX3485 A/B"
- board text removed: "MODULE: BAUTEILSEITE OBEN"
- board text removed: "PGND NIE AN GND"
- board text removed: "PIN 1 = ECKIGES PAD"
- board text removed: "R11 R12 NICHT BESTUECKEN"
- board text removed: "ZELLE 18650"
- board text removed: "ZUM WAZISENSE"

Commit message: checked before order PCB
Parts:
- removed D1: SS34, Diode_SMD:D_SMA
- removed J5: I2C_PORT, TerminalBlock_4Ucon:TerminalBlock_4Ucon_1x04_P3.50mm_Vertical
- removed X3: PROBE1, TerminalBlock_4Ucon:TerminalBlock_4Ucon_1x04_P3.50mm_Vertical
- removed X4: PROBE2, TerminalBlock_4Ucon:TerminalBlock_4Ucon_1x04_P3.50mm_Vertical
- added J5A: I2C_PORT, KijaniSpace:TerminalBlock_KF350_1x02, F.Cu at (88.0, 27.0)
- added J5B: I2C_PORT, KijaniSpace:TerminalBlock_KF350_1x02, F.Cu at (81.0, 27.0)
- added Q5: AO3401A, Package_TO_SOT_SMD:SOT-23, F.Cu at (52.0, 38.0)
- added R13: 100k, Resistor_SMD:R_0603_1608Metric, F.Cu at (52.0, 41.5)
- added X3A: PROBE1, KijaniSpace:TerminalBlock_KF350_1x02, F.Cu at (46.0, 113.0)
- added X3B: PROBE1, KijaniSpace:TerminalBlock_KF350_1x02, F.Cu at (53.0, 113.0)
- added X4A: PROBE2, KijaniSpace:TerminalBlock_KF350_1x02, F.Cu at (65.0, 113.0)
- added X4B: PROBE2, KijaniSpace:TerminalBlock_KF350_1x02, F.Cu at (72.0, 113.0)
- C1: footprint Capacitor_THT:CP_Radial_D8.0mm_P3.50mm -> Capacitor_THT:CP_Radial_D5.0mm_P2.00mm
Routing:
- net +VBATT: track 218.9 -> 223.0 mm
- net VB2: track 19.9 -> 16.9 mm
- net Q5_G: track 0.00 -> 2.66 mm
Other:
- board text added: "BLOCKS EACH, GANGED (REV C)"
- board text added: "J5/X3/X4 ARE TWO 2-POLE"
- board text added: "KIJANISPACE CARRIER Rev C"
- board text added: "Q5 = IDEAL DIODE, NOT A"
- board text added: "SCHOTTKY. REV A HAD D1 HERE."
- board text removed: "KIJANISPACE CARRIER Rev A"

Commit message: converted guides, refined scripts, changed pcb-layout, License, calibration via LoRa
Other:
- board text removed: "BLOCKS EACH, GANGED (REV C)"
- board text removed: "J5/X3/X4 ARE TWO 2-POLE"
- board text removed: "J6 = POWER OUT TO WAZISENSE"
- board text removed: "X1 = 18650 CELL IN"
Changed lines of the file:
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@@
 		(tags "THT Terminal Block 4Ucon ItemNo. 10693 vertical pitch 3.5mm size 8x8.3mm drill 1.3mm pad 2.6mm")
 		(property "Reference" "J8"
-			(at 1.75 -4.82 0)
+			(at 8.6 0 0)
+			(unlocked yes)
 			(layer "F.SilkS")
 			(effects
@@
 		(descr "KF350-3.5-2P screw terminal, 3.50 mm. Gangable: place two 7.00 mm apart and the four pads land on the 3.50 mm grid of a 4-pole part.")
 		(property "Reference" "X4A"
-			(at 0 -9.5 0)
+			(at 1.75 -5.8 0)
+			(unlocked yes)
 			(layer "F.SilkS")
 			(effects
@@
 		(duplicate_pad_numbers_are_jumpers no)
 		(fp_line
-			(start -1.75 -4.7)
-			(end 5.25 -4.7)
+			(start -1.75 -3.45)
+			(end 5.25 -3.45)
 			(stroke
 				(width 0.12)
@@
 		)
 		(fp_line
-			(start -1.75 4.7)
-			(end -1.75 -4.7)
+			(start -1.75 3.45)
+			(end -1.75 -3.45)
 			(stroke
 				(width 0.12)
@@
 		)
 		(fp_line
-			(start 5.25 -4.7)
-			(end 5.25 4.7)
+			(start 5.25 -3.45)
+			(end 5.25 3.45)
 			(stroke
 				(width 0.12)
@@
 		)
 		(fp_line
-			(start 5.25 4.7)
-			(end -1.75 4.7)
+			(start 5.25 3.45)
+			(end -1.75 3.45)
 			(stroke
 				(width 0.12)
@@
 		(descr "KF350-3.5-2P screw terminal, 3.50 mm. Gangable: place two 7.00 mm apart and the four pads land on the 3.50 mm grid of a 4-pole part.")
 		(property "Reference" "X3B"
-			(at 0 -9.5 0)
+			(at 1.75 -5.8 0)
+			(unlocked yes)
 			(layer "F.SilkS")
 			(effects
@@
 		(duplicate_pad_numbers_are_jumpers no)
 		(fp_line
-			(start -1.75 -4.7)
-			(end 5.25 -4.7)
+			(start -1.75 -3.45)
+			(end 5.25 -3.45)
 			(stroke
 				(width 0.12)
@@
 		)
 		(fp_line
-			(start -1.75 4.7)
-			(end -1.75 -4.7)
+			(start -1.75 3.45)
+			(end -1.75 -3.45)
 			(stroke
 				(width 0.12)
@@
 		)
 		(fp_line
-			(start 5.25 -4.7)
-			(end 5.25 4.7)
+			(start 5.25 -3.45)
+			(end 5.25 3.45)
 			(stroke
 				(width 0.12)
@@
 		)
 		(fp_line
-			(start 5.25 4.7)
-			(end -1.75 4.7)
+			(start 5.25 3.45)
+			(end -1.75 3.45)
 			(stroke
 				(width 0.12)
@@
 		(tags "CP Radial series Radial pin pitch 2.00mm diameter 5mm height 7mm Electrolytic Capacitor")
 		(property "Reference" "C1"
-			(at 1.75 6 0)
+			(at 5.4 0 0)
 			(unlocked yes)
 			(layer "F.SilkS")
@@
 		(duplicate_pad_numbers_are_jumpers no)
 		(fp_line
-			(start 5.25 4.7)
-			(end -1.75 4.7)
+			(start 5.25 3.45)
+			(end -1.75 3.45)
 			(stroke
 				(width 0.12)
@@
 		)
 		(fp_line
-			(start 5.25 -4.7)
-			(end 5.25 4.7)
+			(start 5.25 -3.45)
+			(end 5.25 3.45)
 			(stroke
 				(width 0.12)
@@
 		)
 		(fp_line
-			(start -1.75 4.7)
-			(end -1.75 -4.7)
+			(start -1.75 3.45)
+			(end -1.75 -3.45)
 			(stroke
 				(width 0.12)
@@
 		)
 		(fp_line
-			(start -1.75 -4.7)
-			(end 5.25 -4.7)
+			(start -1.75 -3.45)
+			(end 5.25 -3.45)
 			(stroke
 				(width 0.12)
@@
 		)
 		(fp_text user "1:VCC"
-			(at -14.4 0 0)
+			(at -8 0 0)
 			(layer "F.SilkS")
 			(effects
@@
 		(descr "KF350-3.5-2P screw terminal, 3.50 mm. Gangable: place two 7.00 mm apart and the four pads land on the 3.50 mm grid of a 4-pole part.")
 		(property "Reference" "X3A"
-			(at 0 -9.5 0)
+			(at 1.75 -5.8 0)
+			(unlocked yes)
 			(layer "F.SilkS")
 			(effects
@@
 		(duplicate_pad_numbers_are_jumpers no)
 		(fp_line
-			(start -1.75 -4.7)
-			(end 5.25 -4.7)
+			(start -1.75 -3.45)
+			(end 5.25 -3.45)
 			(stroke
 				(width 0.12)
@@
 		)
 		(fp_line
-			(start -1.75 4.7)
-			(end -1.75 -4.7)
+			(start -1.75 3.45)
+			(end -1.75 -3.45)
 			(stroke
 				(width 0.12)
@@
 		)
 		(fp_line
-			(start 5.25 -4.7)
-			(end 5.25 4.7)
+			(start 5.25 -3.45)
+			(end 5.25 3.45)
 			(stroke
 				(width 0.12)
@@
 		)
 		(fp_line
-			(start 5.25 4.7)
-			(end -1.75 4.7)
+			(start 5.25 3.45)
+			(end -1.75 3.45)
 			(stroke
 				(width 0.12)
@@
 		(tags "SOT TO_SOT_SMD")
 		(property "Reference" "Q5"
-			(at 0 -2.4 0)
+			(at 0 2.8 0)
+			(unlocked yes)
 			(layer "F.SilkS")
 			(effects
@@
 		(tags "resistor")
 		(property "Reference" "R13"
-			(at 0 -1.43 0)
+			(at 0 2.6 0)
+			(unlocked yes)
 			(layer "F.SilkS")
 			(effects
@@
 		(descr "KF350-3.5-2P screw terminal, 3.50 mm. Gangable: place two 7.00 mm apart and the four pads land on the 3.50 mm grid of a 4-pole part.")
 		(property "Reference" "X4B"
-			(at 0 -9.5 0)
+			(at 1.75 -5.8 0)
+			(unlocked yes)
 			(layer "F.SilkS")
 			(effects
@@
 		(duplicate_pad_numbers_are_jumpers no)
 		(fp_line
-			(start -1.75 -4.7)
-			(end 5.25 -4.7)
+			(start -1.75 -3.45)
+			(end 5.25 -3.45)
 			(stroke
 				(width 0.12)
@@
 		)
 		(fp_line
-			(start -1.75 4.7)
-			(end -1.75 -4.7)
+			(start -1.75 3.45)
+			(end -1.75 -3.45)
 			(stroke
 				(width 0.12)
@@
 		)
 		(fp_line
-			(start 5.25 -4.7)
-			(end 5.25 4.7)
+			(start 5.25 -3.45)
+			(end 5.25 3.45)
 			(stroke
 				(width 0.12)
@@
 		)
 		(fp_line
-			(start 5.25 4.7)
-			(end -1.75 4.7)
+			(start 5.25 3.45)
+			(end -1.75 3.45)
 			(stroke
 				(width 0.12)
@@
 		(duplicate_pad_numbers_are_jumpers no)
 		(fp_line
-			(start 5.25 4.7)
-			(end -1.75 4.7)
+			(start 5.25 3.45)
+			(end -1.75 3.45)
 			(stroke
 				(width 0.12)
@@
 		)
 		(fp_line
-			(start 5.25 -4.7)
-			(end 5.25 4.7)
+			(start 5.25 -3.45)
+			(end 5.25 3.45)
 			(stroke
 				(width 0.12)
@@
 		)
 		(fp_line
-			(start -1.75 4.7)
-			(end -1.75 -4.7)
+			(start -1.75 3.45)
+			(end -1.75 -3.45)
 			(stroke
 				(width 0.12)
@@
 		)
 		(fp_line
-			(start -1.75 -4.7)
-			(end 5.25 -4.7)
+			(start -1.75 -3.45)
+			(end 5.25 -3.45)
 			(stroke
 				(width 0.12)
@@
 		(tags "SOT TO_SOT_SMD")
 		(property "Reference" "Q4"
-			(at 3.2 -7.5 0)
+			(at 3.1 0 0)
 			(unlocked yes)
 			(layer "F.SilkS")
@@
 		)
 	)
-	(gr_text "X1 = 18650 CELL IN"
-		(at 93.5 43.25 0)
-		(layer "F.SilkS")
-		(effects
-			(font
-				(size 0.9 0.9)
-				(thickness 0.15)
-			)
-			(justify left)
-		)
-	)
-	(gr_text "J6 = POWER OUT TO WAZISENSE"
-		(at 93.5 44.7 0)
-		(layer "F.SilkS")
-		(effects
-			(font
-				(size 0.9 0.9)
-				(thickness 0.15)
-			)
-			(justify left)
-		)
-	)
 	(gr_text "D6- IS NOT GND - KEEP APART"
-		(at 93.5 46.9 0)
+		(at 93.5 44 0)
 		(layer "F.SilkS")
 		(effects
@@
 	)
 	(gr_text "Q5 = IDEAL DIODE, NOT A"
-		(at 93.5 49.1 0)
+		(at 93.5 46.2 0)
 		(layer "F.SilkS")
 		(effects
@@
 	)
 	(gr_text "SCHOTTKY. REV A HAD D1 HERE."
-		(at 93.5 50.55 0)
-		(layer "F.SilkS")
-		(effects
-			(font
-				(size 0.9 0.9)
-				(thickness 0.15)
-			)
-			(justify left)
-		)
-	)
-	(gr_text "J5/X3/X4 ARE TWO 2-POLE"
-		(at 93.5 52.75 0)
-		(layer "F.SilkS")
-		(effects
-			(font
-				(size 0.9 0.9)
-				(thickness 0.15)
-			)
-			(justify left)
-		)
-	)
-	(gr_text "BLOCKS EACH, GANGED (REV C)"
-		(at 93.5 54.2 0)
+		(at 93.5 47.65 0)
 		(layer "F.SilkS")
 		(effects
@@
 	)
 	(gr_text "LEAVE OPEN, DO NOT BRIDGE:"
-		(at 93.5 56.4 0)
+		(at 93.5 49.85 0)
 		(layer "F.SilkS")
 		(effects
@@
 	)
 	(gr_text "R11 R12 U2 (JP1 REPLACES U2)"
-		(at 93.5 57.85 0)
+		(at 93.5 51.3 0)
 		(layer "F.SilkS")
 		(effects
@@
 	)
 	(gr_text "MODULES: PIN1 = SQUARE PAD"
-		(at 93.5 60.05 0)
+		(at 93.5 53.5 0)
 		(layer "F.SilkS")
 		(effects
@@
 		(layer "F.SilkS")
 		(effects
-			(font
-				(size 1.1 1.1)
-				(thickness 0.15)
-			)
-		)
-	)
-	(gr_text "+"
-		(at 42 42.3 0)
-		(layer "F.SilkS")
-		(effects
